Commit message: Update robot.urdf.xacro

File: urdf/robot.urdf.xacro (robot description, xacro)
@@ -16,5 +16,5 @@
         <parent link="base_link"/>
         <child link="base_scan"/>
-        <origin xyz="0.0 -0.035 0.171" rpy="0.0 0.0 0.0"/>
+        <origin xyz="-0.035 0.0 0.171" rpy="0.0 0.0 0.0"/>
     </joint>
     <joint name="wheel_right_joint" type="continuous">
